File: PCB/ESP32-C3_Wi-Fi_env_sensor.kicad_pcb (KiCad board)
At the start: 2 copper layers, 63 x 27.9 mm, 34 parts, among them J1 DX07S016JA1R1500, J2 JST S2B-PH-SM4-TB(LF)(SN), Q1 DMP2070UQ, U1 ESP32-C3-MINI-1, U2 AP2112K-3.3, U3 MCP73831-2-OT, U4 BME280

Commit message: Move U2, R5, C4 to make C4 more effective
Parts:
- moved C4 4.09 mm to (135.6, 92.7), turned to 0 degrees
- moved R5 2.12 mm to (136.5, 89.8)
- moved U2 2.12 mm to (133.5, 89.8)
- moved C5 2.12 mm to (129.7, 90.6)
Routing:
- net +3V3: track 60.1 -> 58.2 mm
- net GND: vias 28 -> 29
Other:
- board text added: "Rev 1.1"
- board text removed: "Rev 1.0"
Changed lines of the file:
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@@
   )
   (footprint "Resistor_SMD:R_0603_1608Metric_Pad0.98x0.95mm_HandSolder" (layer "F.Cu")
-    (at 136.84525 91.948 -90)
+    (at 136.5305 89.85 -90)
     (descr "Resistor SMD 0603 (1608 Metric), square (rectangular) end terminal, IPC_7351 nominal with elongated pad for handsoldering. (Body size source: IPC-SM-782 page 72, https://www.pcb-3d.com/wordpress/wp-content/uploads/ipc-sm-782a_amendment_1_and_2.pdf), generated with kicad-footprint-generator")
     (tags "resistor handsolder")
@@
   )
   (footprint "Capacitor_SMD:C_0603_1608Metric_Pad1.08x0.95mm_HandSolder" (layer "F.Cu")
-    (at 138.36925 95.758 -90)
+    (at 135.636 92.71)
     (descr "Capacitor SMD 0603 (1608 Metric), square (rectangular) end terminal, IPC_7351 nominal with elongated pad for handsoldering. (Body size source: IPC-SM-782 page 76, https://www.pcb-3d.com/wordpress/wp-content/uploads/ipc-sm-782a_amendment_1_and_2.pdf), generated with kicad-footprint-generator")
     (tags "capacitor handsolder")
@@
     (property "ki_keywords" "cap capacitor")
     (attr smd)
-    (fp_text reference "C4" (at 0 -1.43 90) (layer "F.SilkS")
-        (effects (font (size 1 1) (thickness 0.15)))
-    )
-    (fp_text value "10uF" (at 0 1.43 90) (layer "F.Fab")
-        (effects (font (size 1 1) (thickness 0.15)))
-    )
-    (fp_text user "${REFERENCE}" (at 0 0 90) (layer "F.Fab")
+    (fp_text reference "C4" (at 2.54 0.508) (layer "F.SilkS")
+        (effects (font (size 1 1) (thickness 0.15)))
+    )
+    (fp_text value "10uF" (at 0 1.43) (layer "F.Fab")
+        (effects (font (size 1 1) (thickness 0.15)))
+    )
+    (fp_text user "${REFERENCE}" (at 0 0) (layer "F.Fab")
         (effects (font (size 0.4 0.4) (thickness 0.06)))
     )
@@
     (fp_line (start 0.8 0.4) (end -0.8 0.4)
       (stroke (width 0.1) (type solid)) (layer "F.Fab"))
-    (pad "1" smd roundrect (at -0.8625 0 270) (size 1.075 0.95) (layers "F.Cu" "F.Paste" "F.Mask") (roundrect_rratio 0.25)
+    (pad "1" smd roundrect (at -0.8625 0) (size 1.075 0.95) (layers "F.Cu" "F.Paste" "F.Mask") (roundrect_rratio 0.25)
       (net 4 "Net-(D1-K)") (pintype "passive"))
-    (pad "2" smd roundrect (at 0.8625 0 270) (size 1.075 0.95) (layers "F.Cu" "F.Paste" "F.Mask") (roundrect_rratio 0.25)
+    (pad "2" smd roundrect (at 0.8625 0) (size 1.075 0.95) (layers "F.Cu" "F.Paste" "F.Mask") (roundrect_rratio 0.25)
       (net 2 "GND") (pintype "passive"))
     (model "${KICAD6_3DMODEL_DIR}/Capacitor_SMD.3dshapes/C_0603_1608Metric.wrl"
@@
   )
   (footprint "Capacitor_SMD:C_0603_1608Metric_Pad1.08x0.95mm_HandSolder" (layer "F.Cu")
-    (at 129.98725 92.71 180)
+    (at 129.6725 90.612 180)
     (descr "Capacitor SMD 0603 (1608 Metric), square (rectangular) end terminal, IPC_7351 nominal with elongated pad for handsoldering. (Body size source: IPC-SM-782 page 76, https://www.pcb-3d.com/wordpress/wp-content/uploads/ipc-sm-782a_amendment_1_and_2.pdf), generated with kicad-footprint-generator")
     (tags "capacitor handsolder")
@@
   )
   (footprint "Package_TO_SOT_SMD:SOT-23-5" (layer "F.Cu")
-    (at 133.79725 91.948 180)
+    (at 133.4825 89.85 180)
     (descr "SOT, 5 Pin (https://www.jedec.org/sites/default/files/docs/Mo-178c.PDF variant AA), generated with kicad-footprint-generator ipc_gullwing_generator.py")
     (tags "SOT TO_SOT_SMD")
@@
     (effects (font (size 1.25 1.25) (thickness 0.15)) (justify left bottom))
   )
-  (gr_text "Rev 1.0" (at 127 78.74) (layer "F.SilkS")
+  (gr_text "Rev 1.1" (at 127 78.74) (layer "F.SilkS")
     (effects (font (size 0.8 0.8) (thickness 0.15) bold) (justify left bottom))
   )
@@
   (segment (start 137.963 80.914) (end 138.613 80.264) (width 0.25) (layer "F.Cu") (net 1))
   (segment (start 138.613 80.264) (end 139.455 80.264) (width 0.25) (layer "F.Cu") (net 1))
-  (segment (start 132.588 86.36) (end 132.588 88.9) (width 0.6) (layer "F.Cu") (net 1))
   (segment (start 132.588 83.312) (end 132.588 86.36) (width 0.6) (layer "F.Cu") (net 1))
   (segment (start 137.405 79.614) (end 137.963 79.614) (width 0.25) (layer "F.Cu") (net 1))
   (segment (start 153.3085 85.09) (end 155.6585 85.09) (width 0.25) (layer "F.Cu") (net 1))
   (segment (start 134.7025 81.1975) (end 135.89 81.1975) (width 0.6) (layer "F.Cu") (net 1))
-  (segment (start 130.84975 90.63825) (end 132.4985 88.9895) (width 0.6) (layer "F.Cu") (net 1))
   (segment (start 136.1735 80.914) (end 135.89 81.1975) (width 0.25) (layer "F.Cu") (net 1))
   (segment (start 139.446 84.079) (end 136.84 84.079) (width 0.25) (layer "F.Cu") (net 1))
@@
   (segment (start 132.588 86.36) (end 144.78 86.36) (width 0.6) (layer "F.Cu") (net 1))
   (segment (start 137.405 80.914) (end 136.1735 80.914) (width 0.25) (layer "F.Cu") (net 1))
-  (segment (start 132.65975 92.898) (end 131.03775 92.898) (width 0.5) (layer "F.Cu") (net 1))
+  (segment (start 132.345 90.8) (end 130.723 90.8) (width 0.5) (layer "F.Cu") (net 1))
   (segment (start 137.405 81.564) (end 137.405 80.914) (width 0.25) (layer "F.Cu") (net 1))
   (segment (start 137.405 80.914) (end 137.963 80.914) (width 0.25) (layer "F.Cu") (net 1))
-  (segment (start 131.03775 92.898) (end 130.84975 92.71) (width 0.5) (layer "F.Cu") (net 1))
+  (segment (start 130.723 90.8) (end 130.535 90.612) (width 0.5) (layer "F.Cu") (net 1))
   (segment (start 132.588 83.312) (end 134.7025 81.1975) (width 0.6) (layer "F.Cu") (net 1))
   (segment (start 140.716 84.079) (end 139.446 84.079) (width 0.25) (layer "F.Cu") (net 1))
-  (segment (start 132.588 88.9) (end 132.4985 88.9895) (width 0.25) (layer "F.Cu") (net 1))
   (segment (start 135.89 83.129) (end 135.89 81.1975) (width 0.25) (layer "F.Cu") (net 1))
-  (segment (start 130.84975 92.71) (end 130.84975 90.63825) (width 0.6) (layer "F.Cu") (net 1))
+  (segment (start 130.535 88.413) (end 132.588 86.36) (width 0.5) (layer "F.Cu") (net 1))
+  (segment (start 130.535 90.612) (end 130.535 88.413) (width 0.5) (layer "F.Cu") (net 1))
   (via (at 144.78 86.36) (size 0.8) (drill 0.4) (layers "F.Cu" "B.Cu") (net 1))
   (via (at 153.924 83.312) (size 0.8) (drill 0.4) (layers "F.Cu" "B.Cu") (net 1))
@@
   (via (at 119.634 88.9) (size 0.8) (drill 0.4) (layers "F.Cu" "B.Cu") (free) (net 2))
   (via (at 151.13 89.662) (size 0.8) (drill 0.4) (layers "F.Cu" "B.Cu") (free) (net 2))
+  (via (at 138.43 89.916) (size 0.8) (drill 0.4) (layers "F.Cu" "B.Cu") (free) (net 2))
   (via (at 131.318 99.314) (size 0.8) (drill 0.4) (layers "F.Cu" "B.Cu") (free) (net 2))
   (via (at 149.606 93.218) (size 0.8) (drill 0.4) (layers "F.Cu" "B.Cu") (free) (net 2))
@@
   (via (at 114.554 87.63) (size 0.8) (drill 0.4) (layers "F.Cu" "B.Cu") (free) (net 2))
   (via (at 157.48 80.518) (size 0.8) (drill 0.4) (layers "F.Cu" "B.Cu") (free) (net 2))
-  (via (at 128.778 90.678) (size 0.8) (drill 0.4) (layers "F.Cu" "B.Cu") (free) (net 2))
+  (via (at 128.46325 88.58) (size 0.8) (drill 0.4) (layers "F.Cu" "B.Cu") (free) (net 2))
   (via (at 146.304 86.614) (size 0.8) (drill 0.4) (layers "F.Cu" "B.Cu") (free) (net 2))
   (via (at 155.194 89.662) (size 0.8) (drill 0.4) (layers "F.Cu" "B.Cu") (free) (net 2))
@@
   (segment (start 146.7 97.902) (end 145.796 97.902) (width 0.25) (layer "F.Cu") (net 3))
   (segment (start 148.262 97.218) (end 147.384 97.218) (width 0.25) (layer "F.Cu") (net 3))
+  (segment (start 134.7735 92.71) (end 134.7735 94.82625) (width 0.6) (layer "F.Cu") (net 4))
+  (segment (start 134.7735 94.82625) (end 134.81325 94.866) (width 0.6) (layer "F.Cu") (net 4))
+  (segment (start 134.62 90.8) (end 136.493 90.8) (width 0.25) (layer "F.Cu") (net 4))
   (segment (start 134.93475 94.7445) (end 134.81325 94.866) (width 0.25) (layer "F.Cu") (net 4))
   (segment (start 132.44875 94.554) (end 134.50125 94.554) (width 0.5) (layer "F.Cu") (net 4))
-  (segment (start 137.60725 93.6225) (end 137.60725 94.1335) (width 0.25) (layer "F.Cu") (net 4))
-  (segment (start 136.84525 92.8605) (end 137.60725 93.6225) (width 0.25) (layer "F.Cu") (net 4))
-  (segment (start 137.60725 94.1335) (end 138.36925 94.8955) (width 0.25) (layer "F.Cu") (net 4))
-  (segment (start 136.80775 92.898) (end 136.84525 92.8605) (width 0.25) (layer "F.Cu") (net 4))
-  (segment (start 134.93475 92.898) (end 136.80775 92.898) (width 0.25) (layer "F.Cu") (net 4))
+  (segment (start 134.62 90.8) (end 134.62 92.5565) (width 0.6) (layer "F.Cu") (net 4))
+  (segment (start 134.62 92.5565) (end 134.7735 92.71) (width 0.6) (layer "F.Cu") (net 4))
   (segment (start 134.50125 94.554) (end 134.81325 94.866) (width 0.5) (layer "F.Cu") (net 4))
-  (segment (start 134.93475 92.898) (end 134.93475 94.7445) (width 0.5) (layer "F.Cu") (net 4))
+  (segment (start 136.493 90.8) (end 136.5305 90.7625) (width 0.25) (layer "F.Cu") (net 4))
   (segment (start 141.8825 91.2895) (end 143.002 91.2895) (width 0.25) (layer "F.Cu") (net 5))
   (segment (start 129.54 95.504) (end 130.57375 95.504) (width 0.4) (layer "F.Cu") (net 5))
@@
   (segment (start 152.146 85.852) (end 152.1135 85.8195) (width 0.25) (layer "F.Cu") (net 15))
   (segment (start 149.7635 85.09) (end 152.1135 85.09) (width 0.25) (layer "F.Cu") (net 15))
-  (segment (start 136.80775 90.998) (end 136.84525 91.0355) (width 0.25) (layer "F.Cu") (net 16))
-  (segment (start 134.93475 90.998) (end 136.80775 90.998) (width 0.25) (layer "F.Cu") (net 16))
+  (segment (start 134.62 88.9) (end 136.493 88.9) (width 0.25) (layer "F.Cu") (net 16))
+  (segment (start 136.493 88.9) (end 136.5305 88.9375) (width 0.25) (layer "F.Cu") (net 16))
   (segment (start 124.997 98.044) (end 124.997 95.71) (width 0.25) (layer "F.Cu") (net 17))
   (segment (start 124.997 95.71) (end 124.979 95.692) (width 0.25) (layer "F.Cu") (net 17))
